Commit message: generate scan pose

File: src/fv_ur_description/urdf/ur3e_with_tool.urdf.xacro (robot description, xacro)
@@ -44,5 +44,5 @@
       <origin xyz="0 0 0.101" rpy="0 0 0"/>
       <geometry>
-        <cylinder radius="0.05" length="0.20"/>
+        <cylinder radius="0.04" length="0.20"/>
       </geometry>
       <material name="grey">
@@ -53,5 +53,5 @@
       <origin xyz="0 0 0.101" rpy="0 0 0"/>
       <geometry>
-        <cylinder radius="0.05" length="0.20"/>
+        <cylinder radius="0.04" length="0.20"/>
       </geometry>
     </collision>
@@ -94,3 +94,28 @@
   </joint>
   <!-- Table end -->
+  <!-- Table -->
+  <!-- 0.5m x 0.5m x 0.3m table -->
+  <link name="ground">
+    <visual>
+      <origin xyz="-0.4 0.0 -0.01" rpy="0 0 0"/>
+      <geometry>
+        <box size="1.0 1.0 0.01"/>
+      </geometry>
+      <material name="brown">
+        <color rgba="0.6 0.4 0.2 1.0"/>
+      </material>
+    </visual>
+    <collision>
+      <origin xyz="-0.4 0.0 -0.01" rpy="0 0 0"/>
+      <geometry>
+        <box size="1.0 1.0 0.01"/>
+      </geometry>
+    </collision>
+  </link>
+  <joint name="ground_joint" type="fixed">
+    <parent link="world"/>
+    <child link="ground"/>
+    <origin xyz="0 0 0" rpy="0 0 0"/>
+  </joint>
+  <!-- Table end -->
 </robot>
